File: output/npn_amplifier.kicad_sch (KiCad schematic)
At the start: 6 parts, among them Q1 BC547

Commit message: fix: update pipelines
Parts:
- removed Q1: BC547, symbol Device:Q_NPN_BCE
- added Q1: BC547, symbol Device:Q_NPN
Connections:
- net GND: now also V1.1 (+); no longer R2.2
- net VIN: now also C1.2; no longer C1.1
- net VOUT: now also Q1.E; no longer R3.2
- net at R1.2: no longer R3.1
- now unconnected: R1.1, R2.1
