File: output/zener_clamp.kicad_sch (KiCad schematic)
At the start: 2 parts

Commit message: general purpose language pipelines that works well for 2 terminal components
Parts:
- removed C1: 220n, symbol Device:C
- added Z1: 5V, symbol Device:D_Zener
Connections:
- net GND: now also Z1.1 (K), Z1.2 (A)
Other:
- title: rc_filter -> zener_clamp
Changed lines of the file:
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@@
   (generator_version "1.0")
   (paper "A4")
-  (title_block (title "rc_filter"))
+  (title_block (title "zener_clamp"))
   (symbol
     (lib_id "Device:R")
@@
     (instances
       (project "schematic"
-        (path "/77dd2b25-75e0-4ca1-b221-e21b1ceede50"
+        (path "/4e1659b4-80b2-4c35-b056-f3db928ac7e2"
           (reference "R1")
           (unit 1)
@@
   )
   (symbol
-    (lib_id "Device:C")
-    (at 175.4 112.7 0)
+    (lib_id "Device:D_Zener")
+    (at 175.4 112.7 90)
     (unit 1)
     (in_bom yes)
     (on_board yes)
-    (property "Reference" "C1"
+    (property "Reference" "Z1"
       (at 177.432 111.7 0)
       (effects (font (size 1.27 1.27)))
     )
-    (property "Value" "220n"
+    (property "Value" "5V"
       (at 173.368 111.7 0)
       (effects (font (size 1.27 1.27)))
@@
     (instances
       (project "schematic"
-        (path "/77dd2b25-75e0-4ca1-b221-e21b1ceede50"
-          (reference "C1")
+        (path "/4e1659b4-80b2-4c35-b056-f3db928ac7e2"
+          (reference "Z1")
           (unit 1)
         )
@@
     (instances
       (project "schematic"
-        (path "/77dd2b25-75e0-4ca1-b221-e21b1ceede50"
+        (path "/4e1659b4-80b2-4c35-b056-f3db928ac7e2"
           (reference "#PWR01")
           (unit 1)
